Commit message: Add individual torpedos, colors have to be added

File: uwsim/data/scenes/scene.urdf (robot description, URDF)
Before this commit: robot scene, 5 links, 4 joints
Links:
- added link green_torpedo, mass 5.273; collision mesh filename=package://arena_setup/meshes/green_torpedo.STL; visual mesh filename=package://arena_setup/meshes/green_torpedo.STL
- added link red_torpedo, mass 5.273; collision mesh filename=package://arena_setup/meshes/red_torpedo.STL; visual mesh filename=package://arena_setup/meshes/red_torpedo.STL
Joints:
- added joint green_torpedo_to_pool: type fixed, parent pool, child green_torpedo, origin xyz=10 8 0 rpy=0 0 0.0
- added joint red_torpedo_to_pool: type fixed, parent pool, child red_torpedo, origin xyz=10 8 0 rpy=0 0 0.0

Commit message: Add color to torpedos

File: uwsim/data/scenes/scene.urdf (robot description, URDF)
Before this commit: robot scene, 7 links, 6 joints
Links:
- removed link torpedo_link
Joints:
- removed joint torpedo_to_pool
- joint red_torpedo_to_pool: origin xyz=10 8 0 rpy=0 0 0.0 -> xyz=10.33 8 0 rpy=0 0 3.141592653589793238

Commit message: Update scene.urdf

File: uwsim/data/scenes/scene.urdf (robot description, URDF)
Before this commit: robot scene, 6 links, 5 joints
Joints:
- joint green_torpedo_to_pool: origin xyz=10 8 0 rpy=0 0 0.0 -> xyz=10 8 4 rpy=0 0 0.0
- joint red_torpedo_to_pool: origin xyz=10.33 8 0 rpy=0 0 3.141592653589793238 -> xyz=10.33 8 4 rpy=0 0 3.141592653589793238
